Commit message: jazzy/sim: sim sensors match the real mounts — front-facing laser, 50 Hz IMU, camera mock off
- <ignition_frame_id> → <gz_frame_id> (Harmonic).
- Laser moved from the pre-remount (-0.12, 0, 0.15, yaw π) to the pose the
  stack's static TF claims, (0.12, 0, 0.20, yaw 0). Otherwise every sim scan
  is misregistered against the Thor's base_link→laser.
- IMU 100 → 50 Hz, the real vesc_driver poll rate.
- ZED2 RGB/depth gz sensors gated behind a new enable_camera_mock arg
  (default false): out of scope and too expensive for the sim host and LAN.

Only active with enable_sensors:=true, which real hardware never sets.

Co-Authored-By: Claude Opus 5.5 <noreply@anthropic.com>

File: src/f1tenth_description/urdf/roboracer.urdf.xacro (robot description, xacro)
@@ -2,12 +2,12 @@
 <!--
   roboracer.urdf.xacro - F1TENTH vehicle description.
-  Ported from msauber_stack/msauber_description (ROS 2 Jazzy + Gazebo Harmonic)
-  to ROS 2 Humble + Gazebo Fortress (ignition-fortress). Key differences vs the
-  source:
+  Ported from msauber_stack/msauber_description; targets ROS 2 Jazzy + Gazebo
+  Harmonic (it went through Humble + Fortress in between). Key differences vs
+  the source:
     * Frames use the canonical F1TENTH names (base_link, laser, imu,
       zed2_camera_link, ...) so the model is a drop-in for f1tenth_bringup and
       f1tenth_perception - NOT the 'sauber_*' prefixed names.
-    * ros2_control hardware is ign_ros2_control/IgnitionSystem (was
-      gz_ros2_control/GazeboSimSystem).
+    * ros2_control hardware is gz_ros2_control/GazeboSimSystem, with the
+      controller_manager reading /sim/robot_description (see ros2_control.xacro).
     * The stereo "front camera" is replaced by a ZED2 mock (RGB + depth +
       camera_info on the zed2 optical frame).
@@ -16,13 +16,16 @@
   Args:
     pkg_share      - absolute path to this package's share dir (for mesh_dir).
-    use_sim        - true to emit the ign_ros2_control gazebo plugin + sensors.
-    enable_sensors - true to include the LiDAR / camera / IMU sensor links.
-    control_config - path to the ros2_control controllers.yaml (f1tenth_sim).
+    use_sim            - true to emit the gz_ros2_control + ground-truth gazebo plugins.
+    enable_sensors     - true to include the LiDAR / camera / IMU sensor links.
+    enable_camera_mock - true to also render the ZED2 RGB + depth gz sensors
+                         (sim only, off by default; see sensors.xacro).
+    control_config     - path to the ros2_control controllers.yaml (f1tenth_sim).
 -->
 <robot xmlns:xacro="http://www.ros.org/wiki/xacro" name="roboracer">
-  <xacro:arg name="pkg_share"      default="$(find f1tenth_description)" />
-  <xacro:arg name="use_sim"        default="true" />
-  <xacro:arg name="enable_sensors" default="true" />
-  <xacro:arg name="control_config" default="" />
+  <xacro:arg name="pkg_share"          default="$(find f1tenth_description)" />
+  <xacro:arg name="use_sim"            default="true" />
+  <xacro:arg name="enable_sensors"     default="true" />
+  <xacro:arg name="enable_camera_mock" default="false" />
+  <xacro:arg name="control_config"     default="" />
   <xacro:property name="pkg_share" value="$(arg pkg_share)" />
   <xacro:property name="mesh_dir"  value="${pkg_share}/meshes" />

File: src/f1tenth_description/urdf/sensors.xacro (robot description, xacro)
@@ -1,21 +1,24 @@
 <?xml version="1.0"?>
 <!--
-  sensors.xacro - sensor links + Gazebo Fortress (ignition) sensor plugins.
+  sensors.xacro - sensor links + Gazebo Harmonic sensor plugins.
   NEW relative to msauber (which had only a stereo "front camera" and no LiDAR/
-  IMU in its URDF). Frame names and mount poses match the real F1TENTH stack
-  (f1tenth_description/launch/description.launch.py's static TF +
-  f1tenth_perception/camera.launch.py's static TF; Phase 9 layout, base_link
-  centered between the axles, 0.07m above the ground):
-    base_link -> laser              @ (-0.12, 0, 0.15), yaw=pi  (Hokuyo, rear-facing)
+  IMU in its URDF). Frame names and mount poses match the real F1TENTH stack:
+    base_link -> laser              @ ( 0.12, 0, 0.20), yaw=0   (Hokuyo, front-facing)
     base_link -> imu                @ ( 0,    0, 0   )          (VESC IMU @ base_link)
     base_link -> zed2_camera_link   @ ( 0.12, 0, 0.15), yaw=0   (ZED2, front-facing)
                  -> zed2_left_camera_frame -> zed2_left_camera_optical_frame
-  laser is mirrored to the camera's position (same distance from base_link, same
-  height, opposite side) but rotated 180deg in yaw so it faces backward while the
-  camera faces forward.
-  Gazebo tags use the Fortress conventions: <ignition_frame_id> (NOT gz_frame_id)
-  and the sensors are rendered by the world's ignition::gazebo::systems::Sensors
-  / ::Imu systems. <gazebo> blocks are ignored by robot_state_publisher, so this
-  file is harmless on the real robot.
+  laser matches description.launch.py's real-hardware static_baselink_to_laser
+  (the front-facing remount; its numbers are ruler-measured placeholders, see
+  that file). The sim must scan from the pose the Thor's TF claims, or every
+  scan is misregistered. imu matches vesc.launch.py's identity base_link->imu.
+  Gazebo tags use the Harmonic conventions: <gz_frame_id> (Fortress spelled it
+  <gz_frame_id>), rendered by the world's gz::sim::systems::Sensors / ::Imu
+  systems. <gazebo> blocks are ignored by robot_state_publisher, so this file is
+  harmless on the real robot. The IMU's gz frame id never reaches the stack:
+  f1tenth_sim's drive_bridge restamps the message with the real driver's empty
+  frame_id (output/sim_port_report.md, D3).
+  The ZED2 camera/depth sensors are only rendered with enable_camera_mock:=true
+  (default false): two 1280x720 streams at 30 Hz cost more than the sim host's
+  GPU and the LAN should carry, and nothing consumes them yet.
 -->
 <robot xmlns:xacro="http://www.ros.org/wiki/xacro" name="roboracer">
@@ -33,11 +36,11 @@
       <parent link="base_link"/>
       <child link="laser"/>
-      <!-- Rear-facing: yaw=pi, mirrored to zed2_camera_joint's position below. -->
-      <origin xyz="-0.12 0.0 0.15" rpy="0 0 ${pi}"/>
+      <!-- Front-facing; same values as description.launch.py's static_baselink_to_laser. -->
+      <origin xyz="0.12 0.0 0.20" rpy="0 0 0"/>
     </joint>
     <gazebo reference="laser">
       <sensor name="hokuyo" type="gpu_lidar">
         <topic>scan</topic>
-        <ignition_frame_id>laser</ignition_frame_id>
+        <gz_frame_id>laser</gz_frame_id>
         <update_rate>40</update_rate>
         <always_on>true</always_on>
@@ -83,6 +86,7 @@
       <sensor name="imu_sensor" type="imu">
         <topic>sensors/imu/raw</topic>
-        <ignition_frame_id>imu</ignition_frame_id>
-        <update_rate>100</update_rate>
+        <gz_frame_id>imu</gz_frame_id>
+        <!-- vesc_driver polls the IMU every 20 ms, so ~50 Hz on the car. -->
+        <update_rate>50</update_rate>
         <always_on>true</always_on>
       </sensor>
@@ -120,8 +124,9 @@
     </joint>
     <!-- RGB + depth sensors. Image headers carry the optical frame id. -->
+    <xacro:if value="$(arg enable_camera_mock)">
     <gazebo reference="zed2_left_camera_frame">
       <sensor name="zed2_rgb" type="camera">
         <topic>zed2/zed_node/rgb/image_rect_color</topic>
-        <ignition_frame_id>zed2_left_camera_optical_frame</ignition_frame_id>
+        <gz_frame_id>zed2_left_camera_optical_frame</gz_frame_id>
         <update_rate>30</update_rate>
         <always_on>true</always_on>
@@ -143,5 +148,5 @@
       <sensor name="zed2_depth" type="depth_camera">
         <topic>zed2/zed_node/depth/depth_registered</topic>
-        <ignition_frame_id>zed2_left_camera_optical_frame</ignition_frame_id>
+        <gz_frame_id>zed2_left_camera_optical_frame</gz_frame_id>
         <update_rate>30</update_rate>
         <always_on>true</always_on>
@@ -162,4 +167,5 @@
       </sensor>
     </gazebo>
+    </xacro:if>
   </xacro:if>
 </robot>
