Commit message: f1tenth_sim: simulated camera pan joint (URDF + mount + VFOV test)
sensors.xacro: with the camera rendering, the ZED mount becomes a pan joint --
base_link -> camera_pan_base (fixed, the pivot) -> zed2_camera_link (revolute
about z, +-0.2618 rad, ~6 rad/s velocity limit = servo speed). At pan=0 this is
bit-identical to the old fixed mount (pivot = old mount, zero translation), so
the whole ZED subtree (incl. the gz camera sensors) just rotates with the joint.
With the camera off the mount stays the single fixed joint (no free revolute).
sim_sensor_mounts.yaml adds camera_pan_pivot (= zed2_camera_link by design).
ros2_control.xacro declares camera_pan_joint (position command + state) when the
camera renders, so gz_ros2_control drives it and joint_state_broadcaster reports
the measured angle.

test_sim_matches_car_config.py: mounts check follows the new pivot/revolute
split (and pins pan=0 identity); the hokuyo-outside-VFOV check now sweeps the
whole +-15 deg pan over all 8 housing corners (worst case ~43.4 deg below, still
~9 deg clear of the 34.3 deg half-VFOV).

Co-Authored-By: Claude Opus 4.8 <noreply@anthropic.com>

File: src/f1tenth_description/urdf/ros2_control.xacro (robot description, xacro)
@@ -60,4 +60,19 @@
       <state_interface name="effort"/>
     </joint>
+    <!-- Camera pan: position command, driven by camera_pan_position_controller
+         (controllers.yaml) from the sim pan bridge. Only present when the camera
+         renders (enable_camera_mock), matching the revolute camera_pan_joint in
+         sensors.xacro; otherwise ros2_control would reference a joint that is
+         not in the URDF. The joint_state_broadcaster reports its measured
+         position on /sim/joint_states, which the bridge relays to
+         /camera_pan/joint_state. Servo speed is the joint's URDF velocity limit
+         (~6 rad/s), so the measured angle lags the command. -->
+    <xacro:if value="$(arg enable_camera_mock)">
+      <joint name="camera_pan_joint">
+        <command_interface name="position"/>
+        <state_interface name="position"/>
+        <state_interface name="velocity"/>
+      </joint>
+    </xacro:if>
   </ros2_control>
   <xacro:if value="$(arg use_sim)">

File: src/f1tenth_description/urdf/sensors.xacro (robot description, xacro)
@@ -37,4 +37,10 @@
   <xacro:property name="zed_xyz"
                   value="${sim_mounts['zed2_camera_link']['xyz'][0]} ${sim_mounts['zed2_camera_link']['xyz'][1]} ${sim_mounts['zed2_camera_link']['xyz'][2]}" />
+  <!-- Camera pan pivot (= zed_xyz by design, so pan=0 is identical to the old
+       fixed mount) and the revolute joint limits: +-15 deg, ~6 rad/s servo. -->
+  <xacro:property name="pan_pivot_xyz"
+                  value="${sim_mounts['camera_pan_pivot']['xyz'][0]} ${sim_mounts['camera_pan_pivot']['xyz'][1]} ${sim_mounts['camera_pan_pivot']['xyz'][2]}" />
+  <xacro:property name="pan_limit"    value="0.2618" />   <!-- +-15 deg [rad] -->
+  <xacro:property name="pan_velocity" value="6.0" />      <!-- servo speed limit [rad/s] -->
   <!-- ===== ZED 2i internal geometry: zed_macro.urdf.xacro, model zed2i
        (zed-ros2-wrapper v5.4.1, the submodule's pinned commit 86171bc) ===== -->
@@ -129,11 +135,39 @@
     <!-- Same links, joints and names as the wrapper's zed_macro for
          camera_name zed2 / camera_model zed2i, so the sim tree is the car's. -->
-    <!-- Mounting point (the threaded hole under the camera) -->
-    <link name="zed2_camera_link"/>
-    <joint name="zed2_camera_joint" type="fixed">
-      <parent link="base_link"/>
-      <child link="zed2_camera_link"/>
-      <origin xyz="${zed_xyz}" rpy="0 0 0"/>
-    </joint>
+    <!-- Camera mount. With the camera rendering (enable_camera_mock) it is a
+         PAN joint: base_link -> camera_pan_base (fixed, the pivot) ->
+         zed2_camera_link (revolute about z = the pan angle). At pan=0 this is
+         the old fixed base_link->zed2_camera_link (pivot = the old mount, zero
+         translation on the revolute), so pan=0 is bit-identical to before. The
+         whole ZED subtree below zed2_camera_link (incl. the gz camera sensors)
+         rotates with the joint, so the rendered image pans; the measured joint
+         angle drives the stack's TF via camera_pan_tf_node. SIM ONLY: on the
+         car the pan is the Pico servo. With the camera off, the mount stays the
+         original single fixed joint (no free revolute to flop). -->
+    <xacro:if value="$(arg enable_camera_mock)">
+      <link name="camera_pan_base"/>
+      <joint name="camera_pan_base_joint" type="fixed">
+        <parent link="base_link"/>
+        <child link="camera_pan_base"/>
+        <origin xyz="${pan_pivot_xyz}" rpy="0 0 0"/>
+      </joint>
+      <link name="zed2_camera_link"/>
+      <joint name="camera_pan_joint" type="revolute">
+        <parent link="camera_pan_base"/>
+        <child link="zed2_camera_link"/>
+        <origin xyz="0 0 0" rpy="0 0 0"/>
+        <axis xyz="0 0 1"/>
+        <limit lower="${-pan_limit}" upper="${pan_limit}" effort="5.0" velocity="${pan_velocity}"/>
+        <dynamics damping="0.05" friction="0.0"/>
+      </joint>
+    </xacro:if>
+    <xacro:unless value="$(arg enable_camera_mock)">
+      <link name="zed2_camera_link"/>
+      <joint name="zed2_camera_joint" type="fixed">
+        <parent link="base_link"/>
+        <child link="zed2_camera_link"/>
+        <origin xyz="${zed_xyz}" rpy="0 0 0"/>
+      </joint>
+    </xacro:unless>
     <link name="zed2_camera_center">
       <inertial><xacro:sensor_inertial_params /></inertial>
