Commit message: snapshot before campaign-final (2026-10-12)
Working state of linus' jazzy checkout as found on 2026-10-12, kept on its
own branch as a safety net before the campaign-final work.

Co-Authored-By: Claude Opus 5.5 <noreply@anthropic.com>

File: src/f1tenth_description/urdf/core.xacro (robot description, xacro)
@@ -1,11 +1,25 @@
 <?xml version="1.0" ?>
 <!--
-  core.xacro - chassis, wheels and steering hinges for the F1TENTH car.
-  Ported from msauber_description/urdf/core.xacro. Link/joint names are the
-  canonical unprefixed F1TENTH names (base_link is the kinematic root).
-  Geometry (wheelbase 0.325 m, track 0.2 m) is kept as-ported from msauber.
+  core.xacro - base_link, chassis, wheels and steering hinges.
+  base_link is the kinematic root: on the ground, at the rear axle, laterally
+  centred. chassis sits at axle height (wheel_radius) above it; the wheel and
+  hinge joints hang off chassis at the axle positions.
+  Link/joint names are the canonical unprefixed F1TENTH names and must not
+  change: ros2_control.xacro, controllers.yaml and the gazebo <reference>
+  friction tags all address them by name.
+  Wheel joint geometry: the wheel meshes (left_wheel.stl / right_wheel.stl,
+  r 0.05, width 0.045, axle along the mesh z) are scaled to wheel_radius /
+  wheel_width. Each extends OUTWARD from its joint, so the joint sits at
+  y = +-(track - wheel_width)/2 and the tyre centre lands on +-track/2.
+  Sign conventions (verified in the sim port, output/sim_port_report.md 2.2):
+  hinge rpy (0, pi/2, 0) with axis -x, so + hinge angle = +yaw (left); wheel
+  rpy (pi/2, 0, 0) with axis -z, so + wheel velocity rolls toward +x.
 -->
 <robot xmlns:xacro="http://www.ros.org/wiki/xacro" name="roboracer">
-  <!-- Kinematic root -->
+  <xacro:property name="wheel_joint_y" value="${(track - wheel_width) / 2.0}" />
+  <xacro:property name="wheel_mesh_scale"
+                  value="${wheel_radius / 0.05} ${wheel_radius / 0.05} ${wheel_width / 0.045}" />
+  <!-- Kinematic root. No base_footprint: base_link is already on the ground,
+       and the stack never uses one (slam_toolbox_params.yaml base_frame). -->
   <link name="base_link"/>
   <link name="chassis">
@@ -14,7 +28,16 @@
       <material name="red" />
     </visual>
+    <!-- Body box (between the wheels) so the car hits walls with its body, not
+         only its tyres. mu = 0 in ros2_control.xacro: it slides, never drives. -->
+    <collision>
+      <origin xyz="${(body_front_x + body_rear_x) / 2.0} 0
+                   ${(body_top + body_bottom) / 2.0 - wheel_radius}" rpy="0 0 0" />
+      <geometry>
+        <box size="${body_front_x - body_rear_x} ${track - wheel_width} ${body_top - body_bottom}" />
+      </geometry>
+    </collision>
   </link>
   <joint name="base_link_joint" type="fixed">
-    <origin xyz="0 0 0.05" rpy="0 0 0" />
+    <origin xyz="0 0 ${wheel_radius}" rpy="0 0 0" />
     <parent link="base_link" />
     <child link="chassis" />
@@ -30,79 +53,63 @@
     <child link="chassis_inertia" />
   </joint>
-  <!-- Left rear wheel (traction) -->
-  <link name="left_rear_wheel">
-    <inertial><xacro:left_wheels_inertial_params /></inertial>
-    <visual><xacro:left_rear_wheel_geometry /><material name="black" /></visual>
-    <collision><xacro:left_wheels_collision_geometry /></collision>
-  </link>
-  <joint name="left_rear_wheel_joint" type="continuous">
-    <origin xyz="0 0.1 0" rpy="1.5708 0 0" />
-    <parent link="chassis" />
-    <child link="left_rear_wheel" />
-    <axis xyz="0 0 -1" />
-    <limit effort="100" velocity="100" />
-  </joint>
-  <!-- Right rear wheel (traction) -->
-  <link name="right_rear_wheel">
-    <inertial><xacro:right_wheels_inertial_params /></inertial>
-    <visual><xacro:right_rear_wheel_geometry /><material name="black" /></visual>
-    <collision><xacro:right_wheels_collision_geometry /></collision>
-  </link>
-  <joint name="right_rear_wheel_joint" type="continuous">
-    <origin xyz="0 -0.1 0" rpy="1.5708 0 0" />
-    <parent link="chassis" />
-    <child link="right_rear_wheel" />
-    <axis xyz="0 0 -1" />
-    <limit effort="100" velocity="100" />
-  </joint>
-  <!-- Left steering hinge -->
-  <link name="left_steering_hinge">
-    <inertial><xacro:steering_hinge_inertial_params /></inertial>
-    <visual><xacro:left_steering_hinge_geometry /><material name="grey" /></visual>
-  </link>
-  <joint name="left_steering_hinge_joint" type="revolute">
-    <origin xyz="0.325 0.1 0" rpy="0 1.5708 0" />
-    <parent link="chassis" />
-    <child link="left_steering_hinge" />
-    <axis xyz="-1 0 0" />
-    <limit lower="-0.4" upper="0.4" effort="10" velocity="10" />
-  </joint>
-  <!-- Right steering hinge -->
-  <link name="right_steering_hinge">
-    <inertial><xacro:steering_hinge_inertial_params /></inertial>
-    <visual><xacro:right_steering_hinge_geometry /><material name="grey" /></visual>
-  </link>
-  <joint name="right_steering_hinge_joint" type="revolute">
-    <origin xyz="0.325 -0.1 0" rpy="0 1.5708 0" />
-    <parent link="chassis" />
-    <child link="right_steering_hinge" />
-    <axis xyz="-1 0 0" />
-    <limit lower="-0.4" upper="0.4" effort="10" velocity="10" />
-  </joint>
-  <!-- Left front wheel (steered) -->
-  <link name="left_front_wheel">
-    <inertial><xacro:left_wheels_inertial_params /></inertial>
-    <visual><xacro:left_front_wheel_geometry /><material name="black" /></visual>
-    <collision><xacro:left_wheels_collision_geometry /></collision>
-  </link>
-  <joint name="left_front_wheel_joint" type="continuous">
-    <origin xyz="0 0 0" rpy="1.5708 0 0" />
-    <parent link="left_steering_hinge" />
-    <child link="left_front_wheel" />
-    <axis xyz="0 0 -1" />
-    <limit effort="100" velocity="100" />
-  </joint>
-  <!-- Right front wheel (steered) -->
-  <link name="right_front_wheel">
-    <inertial><xacro:right_wheels_inertial_params /></inertial>
-    <visual><xacro:right_front_wheel_geometry /><material name="black" /></visual>
-    <collision><xacro:right_wheels_collision_geometry /></collision>
-  </link>
-  <joint name="right_front_wheel_joint" type="continuous">
-    <origin xyz="0 0 0" rpy="1.5708 0 0" />
-    <parent link="right_steering_hinge" />
-    <child link="right_front_wheel" />
-    <axis xyz="0 0 -1" />
-    <limit effort="100" velocity="100"/>
-  </joint>
+  <!-- One wheel. side: left|right. steer: true -> revolute steering hinge at
+       (x, y) with the wheel on it; false -> wheel directly on the chassis. -->
+  <xacro:macro name="wheel" params="side axle x steer">
+    <xacro:property name="sign" value="${1 if side == 'left' else -1}" />
+    <xacro:property name="y"    value="${sign * wheel_joint_y}" />
+    <!-- left mesh spans z in [-w, 0], right mesh [0, +w]: both point outward -->
+    <xacro:property name="z_off" value="${-sign * wheel_width / 2.0}" />
+    <link name="${side}_${axle}_wheel">
+      <inertial><xacro:wheel_inertial_params z_off="${z_off}" /></inertial>
+      <visual>
+        <origin xyz="0 0 0" rpy="0 0 0" />
+        <geometry>
+          <mesh filename="${mesh_dir}/${side}_wheel.stl" scale="${wheel_mesh_scale}" />
+        </geometry>
+        <material name="black" />
+      </visual>
+      <collision>
+        <origin xyz="0 0 ${z_off}" rpy="0 0 0" />
+        <geometry><cylinder length="${wheel_width}" radius="${wheel_radius}" /></geometry>
+      </collision>
+    </link>
+    <xacro:if value="${steer}">
+      <link name="${side}_steering_hinge">
+        <inertial><xacro:steering_hinge_inertial_params /></inertial>
+        <visual>
+          <origin xyz="0 0 0" rpy="0 0 0" />
+          <geometry><mesh filename="${mesh_dir}/hinge.stl" /></geometry>
+          <material name="grey" />
+        </visual>
+      </link>
+      <joint name="${side}_steering_hinge_joint" type="revolute">
+        <origin xyz="${x} ${y} 0" rpy="0 ${pi/2} 0" />
+        <parent link="chassis" />
+        <child link="${side}_steering_hinge" />
+        <axis xyz="-1 0 0" />
+        <limit lower="${-steer_limit}" upper="${steer_limit}" effort="10" velocity="10" />
+      </joint>
+      <joint name="${side}_${axle}_wheel_joint" type="continuous">
+        <origin xyz="0 0 0" rpy="${pi/2} 0 0" />
+        <parent link="${side}_steering_hinge" />
+        <child link="${side}_${axle}_wheel" />
+        <axis xyz="0 0 -1" />
+        <limit effort="100" velocity="100" />
+      </joint>
+    </xacro:if>
+    <xacro:unless value="${steer}">
+      <joint name="${side}_${axle}_wheel_joint" type="continuous">
+        <origin xyz="${x} ${y} 0" rpy="${pi/2} 0 0" />
+        <parent link="chassis" />
+        <child link="${side}_${axle}_wheel" />
+        <axis xyz="0 0 -1" />
+        <limit effort="100" velocity="100" />
+      </joint>
+    </xacro:unless>
+  </xacro:macro>
+  <!-- Rear axle (traction) at x = 0, front axle (steered) at x = wheelbase -->
+  <xacro:wheel side="left"  axle="rear"  x="0"            steer="false" />
+  <xacro:wheel side="right" axle="rear"  x="0"            steer="false" />
+  <xacro:wheel side="left"  axle="front" x="${wheelbase}" steer="true"  />
+  <xacro:wheel side="right" axle="front" x="${wheelbase}" steer="true"  />
 </robot>

File: src/f1tenth_description/urdf/macros.xacro (robot description, xacro)
@@ -1,8 +1,8 @@
 <?xml version="1.0"?>
 <!--
-  macros.xacro - materials, inertial/geometry macros for the F1TENTH model.
-  Ported verbatim (geometry + inertials) from msauber_description/urdf/macros.xacro;
-  gazebo-classic transmission macros were dropped (gz_ros2_control does not use
-  <transmission> tags).
+  macros.xacro - materials, inertia helpers and the body-mesh fit.
+  Everything is derived from the single-source dimensions in
+  roboracer.urdf.xacro (wheelbase, track, wheel_radius, wheel_width,
+  body_bottom, body_top, body_width). Nothing here hardcodes a vehicle size.
 -->
 <robot name="roboracer" xmlns:xacro="http://www.ros.org/wiki/xacro">
@@ -12,28 +12,70 @@
   <material name="green"><color rgba="0.0 0.8 0.0 1.0"/></material>
   <material name="grey"><color rgba="0.2 0.2 0.2 1.0"/></material>
+  <material name="dark_grey"><color rgba="0.25 0.25 0.25 1.0"/></material>
   <material name="orange"><color rgba="${255/255} ${108/255} ${10/255} 1.0"/></material>
   <material name="red"><color rgba="0.8 0.0 0.0 1.0"/></material>
   <material name="white"><color rgba="1.0 1.0 1.0 1.0"/></material>
-  <!-- inertial parameter macros -->
+  <!-- ====================== body mesh (chassis.stl) ====================== -->
+  <!-- The msauber shell, in millimetres, with its own axes: X runs rear->front
+       NEGATIVE (rear hub at X=465.0, front hub at X=140.0, so its own wheelbase
+       is 325 mm), Y is up (hub centres at Y=192.42, shell Y 161.58..359.91),
+       Z is lateral (3.73..288.73, centre 146.23). Measured from the STL.
+       The fit below puts both hubs on the URDF axles and scales the shell into
+       the F1TENTH envelope: length by wheelbase, width to body_width, and
+       height to body_bottom..body_top (the hub ring then sits ~5 mm above the
+       axle, invisible behind the wheel). rpy (pi/2, 0, pi) maps mesh
+       (X, Y, Z) to car (-x, z, y). -->
+  <xacro:property name="mesh_rear_hub_x"  value="465.0" />
+  <xacro:property name="mesh_hub_dist"    value="325.0" />
+  <xacro:property name="mesh_y_min"       value="161.582" />
+  <xacro:property name="mesh_y_max"       value="359.914" />
+  <xacro:property name="mesh_z_centre"    value="146.2256" />
+  <xacro:property name="mesh_z_width"     value="285.0" />
+  <xacro:property name="body_sx" value="${wheelbase / mesh_hub_dist}" />
+  <xacro:property name="body_sy" value="${(body_top - body_bottom) / (mesh_y_max - mesh_y_min)}" />
+  <xacro:property name="body_sz" value="${body_width / mesh_z_width}" />
+  <!-- Body extents in base_link (x from the rear axle). Used for the collision
+       box; swept_clearance_body_*_x_m in stack_params.yaml describe the same
+       footprint for the car. -->
+  <xacro:property name="body_front_x" value="${(mesh_rear_hub_x - 17.508) * body_sx}" />
+  <xacro:property name="body_rear_x"  value="${(mesh_rear_hub_x - 547.254) * body_sx}" />
+  <!-- Visual, in the chassis frame (chassis sits at axle height). -->
+  <xacro:macro name="chassis_geometry">
+    <origin xyz="${mesh_rear_hub_x * body_sx}
+                 ${-mesh_z_centre * body_sz}
+                 ${body_bottom - wheel_radius - mesh_y_min * body_sy}"
+            rpy="${pi/2} 0 ${pi}" />
+    <geometry>
+      <mesh filename="${mesh_dir}/chassis.stl" scale="${body_sx} ${body_sy} ${body_sz}"/>
+    </geometry>
+  </xacro:macro>
+  <!-- ============================ inertials ============================== -->
+  <!-- Masses unchanged from msauber (chassis 4.0 kg, wheel 0.34055 kg, hinge
+       0.1 kg). The chassis CoM sits midway between the axles at the reference
+       CG height (0.074 m, f1tenth_simulator params.yaml), and its inertia is
+       the solid box of the body envelope. -->
+  <xacro:property name="chassis_mass" value="4.0" />
+  <xacro:property name="wheel_mass"   value="0.34055" />
+  <xacro:macro name="box_inertia" params="m x y z">
+    <inertia ixx="${m * (y*y + z*z) / 12.0}" ixy="0" ixz="0"
+             iyy="${m * (x*x + z*z) / 12.0}" iyz="0"
+             izz="${m * (x*x + y*y) / 12.0}" />
+  </xacro:macro>
   <xacro:macro name="chassis_inertial_params">
-    <origin xyz="0.1477 0 0" rpy="0 0 0" />
-    <mass value="4.0" />
-    <inertia ixx="0.010609" ixy="0" ixz="0"
-             iyy="0.050409" iyz="0"
-             izz="0.05865" />
+    <origin xyz="${wheelbase / 2.0} 0 ${0.074 - wheel_radius}" rpy="0 0 0" />
+    <mass value="${chassis_mass}" />
+    <xacro:box_inertia m="${chassis_mass}" x="${body_front_x - body_rear_x}"
+                       y="${body_width}" z="${body_top - body_bottom}" />
   </xacro:macro>
-  <xacro:macro name="left_wheels_inertial_params">
-    <origin xyz="0 0 -0.0225" rpy="0 0 0" />
-    <mass value="0.34055" />
-    <inertia ixx="0.00026046" ixy="0" ixz="0"
-             iyy="0.00026046" iyz="0"
-             izz="0.00041226" />
-  </xacro:macro>
-  <xacro:macro name="right_wheels_inertial_params">
-    <origin xyz="0 0 0.0225" rpy="0 0 0" />
-    <mass value="0.34055" />
-    <inertia ixx="0.00026046" ixy="0" ixz="0"
-             iyy="0.00026046" iyz="0"
-             izz="0.00041226" />
+  <!-- Solid cylinder about its own z (the wheel axle). z_off puts the CoM in
+       the middle of the tyre: the wheel mesh extends outward from the joint. -->
+  <xacro:macro name="wheel_inertial_params" params="z_off">
+    <origin xyz="0 0 ${z_off}" rpy="0 0 0" />
+    <mass value="${wheel_mass}" />
+    <inertia ixx="${wheel_mass * (3*wheel_radius*wheel_radius + wheel_width*wheel_width) / 12.0}"
+             ixy="0" ixz="0"
+             iyy="${wheel_mass * (3*wheel_radius*wheel_radius + wheel_width*wheel_width) / 12.0}"
+             iyz="0"
+             izz="${wheel_mass * wheel_radius * wheel_radius / 2.0}" />
   </xacro:macro>
   <xacro:macro name="steering_hinge_inertial_params">
@@ -52,42 +94,3 @@
              izz="1e-5" />
   </xacro:macro>
-  <!-- geometry macros -->
-  <xacro:macro name="chassis_geometry">
-    <origin xyz="0.46 -0.135 -0.180" rpy="1.57 0 3.14" />
-    <geometry>
-      <mesh filename="${mesh_dir}/chassis.stl" scale="0.000990 0.0009375 0.0009375"/>
-    </geometry>
-  </xacro:macro>
-  <xacro:macro name="left_rear_wheel_geometry">
-    <origin xyz="0 0 0" rpy="0 0 0" />
-    <geometry><mesh filename="${mesh_dir}/left_wheel.stl" /></geometry>
-  </xacro:macro>
-  <xacro:macro name="right_rear_wheel_geometry">
-    <origin xyz="0 0 0" rpy="0 0 0" />
-    <geometry><mesh filename="${mesh_dir}/right_wheel.stl" /></geometry>
-  </xacro:macro>
-  <xacro:macro name="left_front_wheel_geometry">
-    <origin xyz="0 0 0" rpy="0 0 0" />
-    <geometry><mesh filename="${mesh_dir}/left_wheel.stl" /></geometry>
-  </xacro:macro>
-  <xacro:macro name="right_front_wheel_geometry">
-    <origin xyz="0 0 0" rpy="0 0 0" />
-    <geometry><mesh filename="${mesh_dir}/right_wheel.stl" /></geometry>
-  </xacro:macro>
-  <xacro:macro name="left_steering_hinge_geometry">
-    <origin xyz="0 0 0" rpy="0 0 0" />
-    <geometry><mesh filename="${mesh_dir}/hinge.stl" /></geometry>
-  </xacro:macro>
-  <xacro:macro name="right_steering_hinge_geometry">
-    <origin xyz="0 0 0" rpy="0 0 0" />
-    <geometry><mesh filename="${mesh_dir}/hinge.stl" /></geometry>
-  </xacro:macro>
-  <xacro:macro name="left_wheels_collision_geometry">
-    <origin xyz="0 0 -0.0225" rpy="0 0 0" />
-    <geometry><cylinder length="0.045" radius="0.05" /></geometry>
-  </xacro:macro>
-  <xacro:macro name="right_wheels_collision_geometry">
-    <origin xyz="0 0 0.0225" rpy="0 0 0" />
-    <geometry><cylinder length="0.045" radius="0.05" /></geometry>
-  </xacro:macro>
 </robot>

File: src/f1tenth_description/urdf/roboracer.urdf.xacro (robot description, xacro)
@@ -1,23 +1,29 @@
 <?xml version="1.0" ?>
 <!--
-  roboracer.urdf.xacro - F1TENTH vehicle description.
-  Ported from msauber_stack/msauber_description; targets ROS 2 Jazzy + Gazebo
-  Harmonic (it went through Humble + Fortress in between). Key differences vs
-  the source:
-    * Frames use the canonical F1TENTH names (base_link, laser, imu,
-      zed2_camera_link, ...) so the model is a drop-in for f1tenth_bringup and
-      f1tenth_perception - NOT the 'sauber_*' prefixed names.
-    * ros2_control hardware is gz_ros2_control/GazeboSimSystem, with the
-      controller_manager reading /sim/robot_description (see ros2_control.xacro).
-    * The stereo "front camera" is replaced by a ZED2 mock (RGB + depth +
-      camera_info on the zed2 optical frame).
-    * A 2D Hokuyo-like LiDAR (/scan) and an IMU (/sensors/imu/raw) are added
-      (the source had neither in the URDF).
+  roboracer.urdf.xacro - F1TENTH vehicle description (the only top-level model).
+  Used by the stack's robot_state_publisher on the car (description.launch.py,
+  use_sim:=false enable_sensors:=false: body + wheels only) and by f1tenth_sim's
+  private robot_state_publisher (use_sim:=true enable_sensors:=true).
+  Ported from msauber_stack/msauber_description. The body is still the msauber
+  "Sauber" shell mesh, but it is now scaled into the F1TENTH reference envelope
+  below, so the visual, the wheels and the sim physics all have F1TENTH size.
+  ===================== single-source dimensions =====================
+  F1TENTH reference values (f1tenth_simulator racecar.xacro / params.yaml, the
+  same numbers f1tenth_gym uses). The car's own wheelbase has never been
+  measured: vesc.yaml and the MPC use 0.305 (docs/DIAGNOSTICS.md, backlog P2).
+  Every dimension lives here once; core.xacro, sensors.xacro and the sim's
+  controllers.yaml / drive_bridge derive from it (test_sim_matches_car_config.py
+  checks the sim side).
+  base_link: on the ground plane, at the rear axle, laterally centred. That is
+  the point the odometry (vesc_to_odom's bicycle model, the sim's
+  ackermann_steering_controller) integrates, and the frame the EKF drives.
   Args:
-    pkg_share      - absolute path to this package's share dir (for mesh_dir).
+    pkg_share          - absolute path to this package's share dir (for mesh_dir).
     use_sim            - true to emit the gz_ros2_control + ground-truth gazebo plugins.
-    enable_sensors     - true to include the LiDAR / camera / IMU sensor links.
-    enable_camera_mock - true to also render the ZED2 RGB + depth gz sensors
-                         (sim only, off by default; see sensors.xacro).
+    enable_sensors     - true to include the LiDAR / IMU / ZED 2i links. Sim only:
+                         on the car those frames come from static TF publishers
+                         and the ZED wrapper (see description.launch.py).
+    enable_camera_mock - true to also render the ZED 2i RGB + depth gz sensors
+                         (sim only; f1tenth_sim's `camera` arg, default on).
     control_config     - path to the ros2_control controllers.yaml (f1tenth_sim).
 -->
@@ -30,4 +36,15 @@
   <xacro:property name="pkg_share" value="$(arg pkg_share)" />
   <xacro:property name="mesh_dir"  value="${pkg_share}/meshes" />
+  <!-- Wheels and axles (F1TENTH reference). -->
+  <xacro:property name="wheelbase"    value="0.3302" />  <!-- rear axle -> front axle -->
+  <xacro:property name="track"        value="0.2413" />  <!-- wheel centre -> wheel centre -->
+  <xacro:property name="wheel_radius" value="0.0508" />
+  <xacro:property name="wheel_width"  value="0.0381" />
+  <!-- Body envelope (F1TENTH reference: bottom 0.04 m, height 0.1 m). The body
+       is as wide as the outside of the wheels. -->
+  <xacro:property name="body_bottom"  value="0.04" />    <!-- above ground -->
+  <xacro:property name="body_top"     value="0.14" />    <!-- above ground -->
+  <xacro:property name="body_width"   value="${track + wheel_width}" />
+  <xacro:property name="steer_limit"  value="0.4" />     <!-- hinge joint limit [rad] -->
   <xacro:include filename="${pkg_share}/urdf/macros.xacro" />
   <xacro:include filename="${pkg_share}/urdf/core.xacro" />
