Commit message: vehicle frames: bumper, LiDAR and ZED positions from the 2026-10-13 tape measurement
DELIBERATE CHANGE FROM THE FIRST TEST CAMPAIGN, which ran with the old values.

Measured on the car by Andreas, all to the bumper face: front axle centre
0.10 m, LiDAR scan centre 0.10 m, ZED front face 0.15 m. Both static TFs
already hang off base_link (description.launch.py, camera.launch.py), so
nothing is double-counted. base_link stays on the rear axle: it is where
vesc_to_odom.cpp's bicycle integrates (no slip angle) and where core.xacro
puts the rear wheels.

  frame (parent base_link)  old (campaign)  new     how
  base_front  x             0.443           0.425   URDF wheelbase 0.325 + 0.10 (was the chassis-mesh front, never measured)
  laser       x             0.12            0.325   0.425 - 0.10
  zed2_camera_link x        0.12            0.260   0.425 - 0.15 - 0.0151
  (y, z and rotations unchanged: laser 0, 0.20, yaw 0; zed 0, 0.15, yaw 0)

The ZED is a ZED 2i (S/N 36866199, the SDK reports it; the launch still
says camera_model zed2). zed2_camera_link is its mounting screw; zed2i.stl
reaches +0.0251 m from a mesh origin at screw_offset_x -0.01
(zed_macro.urdf.xacro), so the front face is 0.0151 m ahead of it.
The left optical frame moves from x 0.110 to 0.250: lens -> bumper 0.175 m
(was 0.333).

What it moves (all read base_front / the static TFs at runtime):
- every front distance: /perception/front_distance and front_clearance
  (camera, lens offset 0.333 -> 0.175), /costmap/front_clearance,
  /mpc/min_obstacle_distance*, the mission wall stop and wall_turn trigger;
- the e-stop front cone (IsProximityTooClose): laser -> bumper 0.323 -> 0.10;
- SLAM and the costmap: every scan point moves 0.205 m forward in base_link;
- 3D detection positions (detection_3d / obstacle_projector via the ZED TF):
  0.14 m forward;
- go_to gap: gap_min(person) 0.53 -> 0.5475, so a clamped gap is 0.55 (was
  0.53); the 0.6 default is unchanged. Corridor sizing still holds:
  hw(1.425) = 0.874 >= 0.87 with the 0.64 start.

Tests: test_base_front asserts 0.425 (renamed); new test_sensor_extrinsics
(laser = base_front - 0.10) and test_zed_extrinsic (zed = base_front - 0.15 -
0.0151) pin the launch files to the bumper; the go_to tests that encode the
old bumper (front_x 0.443, clamped gap 0.53, ex10 golden regenerated with
translate()) updated. Docstrings that stated 0.443 / 0.12 updated.
Not changed: sensors.xacro (sim only, stale LiDAR pose, backlog B10).

Co-Authored-By: Claude Opus 5.5 (1M context) <noreply@anthropic.com>

File: src/f1tenth_description/urdf/base_front.xacro (robot description, xacro)
@@ -11,11 +11,13 @@
   f1tenth_description.vehicle_frames.base_front_xyz(), which parses THIS FILE's
   base_front_* properties. Do not copy the number anywhere else.
-  x = 0.443 m: the front of the chassis mesh, from base_link at the rear axle
-  (base_link convention: core.xacro / base.xacro). Taken from the URDF chassis
-  mesh bounds, as stack_params' swept_clearance_body_front_x_m was; NOT
-  measured on the car. z = 0: base_link's own plane.
+  x = 0.425 m (2026-10-13, MEASURED): base_link is the rear axle (core.xacro,
+  and the odometry's rear-axle bicycle in vesc_to_odom.cpp); the URDF wheelbase
+  is 0.325 m (core.xacro steering hinges) and Andreas taped front axle centre ->
+  bumper face = 0.10 m on the car, so 0.325 + 0.10. Until then it was 0.443, the
+  front of the chassis mesh, never measured; the first test campaign ran with
+  0.443. z = 0: base_link's own plane.
 -->
 <robot xmlns:xacro="http://www.ros.org/wiki/xacro">
-  <xacro:property name="base_front_x" value="0.443" />
+  <xacro:property name="base_front_x" value="0.425" />
   <xacro:property name="base_front_y" value="0.0" />
   <xacro:property name="base_front_z" value="0.0" />

Commit message: vehicle frames: wheelbase 0.305 in the URDF; bumper, LiDAR and ZED follow
DELIBERATE CHANGE FROM THE FIRST TEST CAMPAIGN (and corrects bdc7c93's
use of the URDF's 0.325). Andreas, 2026-10-13: the wheelbase is 0.305, as
odometry (vesc.yaml wheelbase) and the MPC (mpc_wheelbase_m) already use;
the URDF's 0.325 (msauber's port) is wrong. Odometry and MPC unchanged.

  value                          campaign   bdc7c93   now
  URDF wheelbase (core.xacro hinges, robot.urdf.xacro)
                                 0.325      0.325     0.305
  base_front x                   0.443      0.425     0.405   = 0.305 + 0.10 taped
  laser x                        0.12       0.325     0.305   = 0.405 - 0.10 taped
  zed2_camera_link x             0.12       0.260     0.2399  = 0.405 - 0.15 - 0.0151
  (left optical frame x)         0.110      0.250     0.2299  lens -> bumper 0.175

What moves vs bdc7c93: every front distance by 2 cm (bumper back), every
scan point and every camera point 2 cm back in base_link (SLAM, costmap,
3D detections), the e-stop cone's apex 2 cm back (laser -> bumper still
0.10). go_to: gap_min(person) 0.5475 -> 0.5675, a clamped gap 0.55 ->
0.57; the 0.6 default unchanged. Corridor: s = 1.405, hw 0.8706 >= 0.87.

The sim keeps its kinematics matched to its URDF: controllers.yaml,
drive_bridge default and sim_bringup's drive_bridge wheelbase 0.325 ->
0.305.

Tests: test_base_front asserts 0.405 (renamed); test_sensor_extrinsics
and test_zed_extrinsic derive from base_front and pass unchanged; the
go_to tests tied to the bumper (front_x 0.405, clamped gap 0.57, ex10
golden regenerated with translate()) updated. Docstrings and stack_params
descriptions that stated 0.425/0.325 updated.

Co-Authored-By: Claude Opus 5.5 (1M context) <noreply@anthropic.com>

File: src/f1tenth_description/urdf/base_front.xacro (robot description, xacro)
@@ -11,13 +11,13 @@
   f1tenth_description.vehicle_frames.base_front_xyz(), which parses THIS FILE's
   base_front_* properties. Do not copy the number anywhere else.
-  x = 0.425 m (2026-10-13, MEASURED): base_link is the rear axle (core.xacro,
-  and the odometry's rear-axle bicycle in vesc_to_odom.cpp); the URDF wheelbase
-  is 0.325 m (core.xacro steering hinges) and Andreas taped front axle centre ->
-  bumper face = 0.10 m on the car, so 0.325 + 0.10. Until then it was 0.443, the
-  front of the chassis mesh, never measured; the first test campaign ran with
-  0.443. z = 0: base_link's own plane.
+  x = 0.405 m (2026-10-13, MEASURED): base_link is the rear axle (core.xacro,
+  and the odometry's rear-axle bicycle in vesc_to_odom.cpp); the wheelbase is
+  0.305 m (odometry and MPC; core.xacro corrected from 0.325 the same day) and
+  Andreas taped front axle centre -> bumper face = 0.10 m on the car, so
+  0.305 + 0.10. Until then it was 0.443, the front of the chassis mesh, never
+  measured; the first test campaign ran with 0.443. z = 0: base_link's own plane.
 -->
 <robot xmlns:xacro="http://www.ros.org/wiki/xacro">
-  <xacro:property name="base_front_x" value="0.425" />
+  <xacro:property name="base_front_x" value="0.405" />
   <xacro:property name="base_front_y" value="0.0" />
   <xacro:property name="base_front_z" value="0.0" />

File: src/f1tenth_description/urdf/core.xacro (robot description, xacro)
@@ -4,5 +4,7 @@
   Ported from msauber_description/urdf/core.xacro. Link/joint names are the
   canonical unprefixed F1TENTH names (base_link is the kinematic root).
-  Geometry (wheelbase 0.325 m, track 0.2 m) is kept as-ported from msauber.
+  Geometry: track 0.2 m as ported from msauber; wheelbase 0.305 m since
+  2026-10-13 (was msauber's 0.325), the value the car's odometry
+  (vesc.yaml wheelbase) and the MPC (mpc_wheelbase_m) use.
 -->
 <robot xmlns:xacro="http://www.ros.org/wiki/xacro" name="roboracer">
@@ -62,5 +64,5 @@
   </link>
   <joint name="left_steering_hinge_joint" type="revolute">
-    <origin xyz="0.325 0.1 0" rpy="0 1.5708 0" />
+    <origin xyz="0.305 0.1 0" rpy="0 1.5708 0" />
     <parent link="chassis" />
     <child link="left_steering_hinge" />
@@ -74,5 +76,5 @@
   </link>
   <joint name="right_steering_hinge_joint" type="revolute">
-    <origin xyz="0.325 -0.1 0" rpy="0 1.5708 0" />
+    <origin xyz="0.305 -0.1 0" rpy="0 1.5708 0" />
     <parent link="chassis" />
     <child link="right_steering_hinge" />

File: src/f1tenth_description/urdf/robot.urdf.xacro (robot description, xacro)
@@ -31,5 +31,5 @@
   <!-- ===================== single-source dimensions ===================== -->
   <!-- Shared with the odometry kinematics (vesc.yaml / drive_bridge wheelbase). -->
-  <xacro:property name="wheelbase"    value="0.325" />  <!-- rear axle -> front axle -->
+  <xacro:property name="wheelbase"    value="0.305" />  <!-- rear axle -> front axle -->
   <xacro:property name="track"        value="0.2"   />  <!-- left wheel -> right wheel -->
   <xacro:property name="wheel_radius" value="0.05"  />
